File: masonjar.kicad_pcb (KiCad board)
At the start: 2 copper layers, 63.8 x 100 mm, 189 parts, among them U1 ESP32-WROOM-32

Commit message: working on layout
Parts:
- moved C32 118.5 mm to (-25.2, 98.0), turned to 315 degrees
- moved C47 113.0 mm to (-18.1, 98.0), turned to 315 degrees
- moved C46 103.7 mm to (-1.73, 106.2)
- moved C33 103.7 mm to (1.18, 108.2)
- moved C36 103.7 mm to (1.18, 106.2)
- moved C37 103.7 mm to (4.09, 104.2)
- moved C40 103.7 mm to (1.18, 104.2)
- moved C41 103.7 mm to (4.09, 106.2)
- moved C35 101.7 mm to (-25.3, 85.5), turned to 315 degrees
- moved C44 97.9 mm to (-18.1, 85.5), turned to 315 degrees
- moved C45 92.2 mm to (-10.8, 85.5), turned to 315 degrees
- moved C34 87.5 mm to (-3.60, 85.5), turned to 315 degrees
- moved R58 87.0 mm to (-3.55, 99.3), turned to 180 degrees
- moved C30 82.2 mm to (3.70, 85.5), turned to 315 degrees
- moved R59 78.2 mm to (3.70, 99.3), turned to 180 degrees
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
Commit message: working on layout
Parts:
- moved C33 26.3 mm to (25.4, 98.0), turned to 315 degrees
- moved C36 18.9 mm to (18.2, 98.0), turned to 315 degrees
- moved C40 13.5 mm to (-10.8, 98.0), turned to 315 degrees
- moved C41 10.6 mm to (10.9, 98.0), turned to 315 degrees
- moved C46 8.32 mm to (-3.55, 98.0), turned to 315 degrees
- moved C37 6.14 mm to (3.70, 98.0), turned to 315 degrees
- moved C44 0.10 mm to (-18.1, 85.5)
- moved C47 0.05 mm to (-18.1, 98.0)
- moved C34 0.05 mm to (-3.55, 85.5)
Routing:
- net GND: track 15.3 -> 19.9 mm, vias 26 -> 72
- net Net-(D35-Pad2): track 0.00 -> 1.45 mm
- net Net-(D34-Pad2): track 0.00 -> 1.45 mm
- net Net-(D29-Pad2): track 0.00 -> 1.45 mm
- net Net-(D28-Pad2): track 0.00 -> 1.45 mm
- net Net-(D33-Pad2): track 0.00 -> 1.45 mm
- net Net-(D32-Pad2): track 0.00 -> 1.45 mm
- net Net-(D31-Pad2): track 0.00 -> 1.45 mm
- net Net-(D62-Pad2): track 0.00 -> 1.45 mm
- net Net-(D61-Pad2): track 0.00 -> 1.45 mm
- net Net-(D56-Pad2): track 0.00 -> 1.45 mm
- net Net-(D55-Pad2): track 0.00 -> 1.45 mm
- net Net-(D53-Pad2): track 0.00 -> 1.45 mm
- net Net-(D52-Pad2): track 0.00 -> 1.45 mm
- net Net-(D47-Pad2): track 0.00 -> 1.45 mm
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
Commit message: working on layout
Parts:
- moved C57 0.16 mm to (-18.1, 60.5)
- moved C58 0.07 mm to (-3.55, 60.5)
- moved C15 0.05 mm to (-18.1, 73.0)
- moved C60 0.05 mm to (25.4, 60.5)
- moved C62 0.05 mm to (-3.55, 73.0)
Routing:
- net +5V: track 346.7 -> 396.2 mm
- net GND: track 19.9 -> 55.5 mm, vias 72 -> 73
- net Net-(D30-Pad2): track 0.00 -> 1.45 mm
- net Net-(D31-Pad4): track 0.00 -> 1.40 mm

Commit message: working on layout
Parts:
- moved C11 69.9 mm to (52.0, -0.61)
- moved C38 69.9 mm to (55.2, 8.64)
- moved C39 69.9 mm to (52.3, 8.64)
- moved C48 69.9 mm to (49.4, 8.64)
- moved C49 69.9 mm to (46.5, 8.64)
- moved C53 69.9 mm to (52.0, 1.38)
- moved C4 46.6 mm to (-5.85, 22.2), turned to 180 degrees
- moved C2 42.7 mm to (0.05, 22.2), turned to 180 degrees
- moved C7 38.1 mm to (7.30, 22.2), turned to 180 degrees
- moved C3 33.5 mm to (14.6, 22.2), turned to 180 degrees
- moved C5 29.7 mm to (21.8, 22.2), turned to 180 degrees
- moved C6 27.0 mm to (29.1, 22.2), turned to 180 degrees
- moved R1 0.28 mm to (-25.3, 23.9)
- moved R3 0.25 mm to (-10.8, 23.9)
- moved R4 0.25 mm to (-3.60, 23.9)
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Routing:
- net +5V: track 396.2 -> 465.8 mm, vias 32 -> 28
- net Net-(D7-Pad4): track 0.00 -> 1.98 mm
- net Net-(D1-Pad2): track 0.00 -> 1.97 mm
- net Net-(D9-Pad4): track 0.00 -> 1.95 mm
- net Net-(D8-Pad4): track 0.00 -> 1.93 mm
- net Net-(D3-Pad4): track 0.00 -> 1.93 mm
- net Net-(D5-Pad4): track 0.00 -> 1.93 mm
- net Net-(D6-Pad4): track 0.00 -> 1.93 mm
- net Net-(D4-Pad4): track 0.00 -> 1.93 mm
- net Net-(D7-Pad2): track 0.00 -> 1.92 mm
- net Net-(D3-Pad2): track 0.00 -> 1.92 mm
- net Net-(D2-Pad2): track 0.00 -> 1.92 mm
- net Net-(D5-Pad2): track 0.00 -> 1.92 mm
- net Net-(D4-Pad2): track 0.00 -> 1.92 mm
- net Net-(D8-Pad2): track 0.00 -> 1.90 mm
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