File: hw/masonjar.sch (KiCad schematic (older format))
At the start: 189 parts, among them U1 ESP32-WROOM-32

Commit message: first fire animation with hue integration
Parts:
- added C64, C65, C66, C68, C69: 100n, Capacitor_SMD:C_0402_1005Metric, symbol Device:C_Small
- added C67, C71, C72, C73, C74: 10u, Capacitor_SMD:C_0805_2012Metric, symbol Device:C_Small
- added C70: 10n, Capacitor_SMD:C_0603_1608Metric, symbol Device:C_Small
- added D64, D65: SS34, Diode_SMD:D_SMA, symbol Device:D_Small
- added J1, J2: Conn_01x05, Connector_PinHeader_2.54mm:PinHeader_1x05_P2.54mm_Vertical, symbol Connector_Generic:Conn_01x05
- added L1: MWSA0402-100MT, Inductor_SMD:L_Taiyo-Yuden_MD-4040, symbol Device:L_Small
- added R63: 75, Resistor_SMD:R_0402_1005Metric, symbol Device:R_Small
- added R64, R65, R67, R74, R76, R77: 10k, Resistor_SMD:R_0402_1005Metric, symbol Device:R_Small
- added R66: R_PHOTO, LED_SMD:LED_0805_2012Metric, symbol Device:R_PHOTO
- added R68: 1M, Resistor_SMD:R_0402_1005Metric, symbol Device:R_Small
- added R69, R70: 1k, Resistor_SMD:R_0402_1005Metric, symbol Device:R_Small
- added R72, R73, R75, R78, R80: 100k, Resistor_SMD:R_0402_1005Metric, symbol Device:R_Small
- added R79: 22k, Resistor_SMD:R_0402_1005Metric, symbol Device:R_Small
- added SW1, SW2: SW_Push_Dual, Button_Switch_SMD:SW_Push_1P1T_NO_6x6mm_H9.5mm, symbol Switch:SW_Push_Dual
- added U2: E75-2G4M20S, footprimt:E75-2G4M10S, symbol masonjar-rescue:E75-2G4M20S-e75-2g4m20s
- added U3: MP2359DJ-LF-Z_[C14259], Package_TO_SOT_SMD:SOT-23-6, symbol masonjar-rescue:MP2359DJ-LF-Z_[C14259]-lc_IC
- gave numbers to parts that had none: 162
Connections:
- net +5V: now also C73.2, C74.2, D64.2 (A), R80.2, U3.5 (IN); no longer D1.1 (VDD)
- net GND: now also U1.1 (GND), U1.15 (GND), U1.38 (GND), C64.2, C65.1, C66.1, C67.1, C68.1, C69.1, C71.1, C72.1, C73.1, C74.1, D65.2 (A), J1.1 (Pin_1), J2.1 (Pin_1), R67.2, R68.1, R79.2, SW1.1, SW1.3, SW2.1, SW2.3, U2.18 (GND), U3.2 (GND)
- net at D1.4 (DIN): now also R63.1
- net +3V3: now reaches U1.2 (VDD)
- net +3V3: now also C67.2, C71.2, C72.2, L1.2, R64.2, R65.2, R66.1, R74.1, R76.1, R77.1, R78.2, U2.17 (VDD)
- net WS2812: now reaches U1.24 (IO2)
- net WS2812: now also R63.2, R67.1
- net at U1.25 (IO0): now also J1.5 (Pin_5), R65.1
- net at U1.27 (IO16): now also R69.2
- net at U1.28 (IO17): now also R70.1
- net EN: now reaches U1.3 (EN)
- net EN: now also J1.4 (Pin_4), R64.1
- net BTN: now reaches U1.33 (IO21)
- net BTN: now also R74.2, SW1.2, SW1.4
- net at U1.34 (RXD0/IO3): now also J1.2 (Pin_2)
- net at U1.35 (TXD0/IO1): now also J1.3 (Pin_3)
- net at U1.5 (SENSOR_VN): now also C65.2, R66.2, R68.2
- net at U1.6 (IO34): now also C69.2, R73.2
- net at U1.7 (IO35): now also C68.2, R75.2
- net at U1.9 (IO33): now also C66.2, R72.2
- new net: C64.1, D1.1 (VDD), D64.1 (K)
- new net: J2.5 (Pin_5), R77.2, U2.3 (SPI_MISO)
- new net: C70.2, U3.1 (BST)
- new net: R78.1, R79.1, U3.3 (FB)
- new net: R80.1, U3.4 (EN)
- new net: C70.1, D65.1 (K), L1.1, U3.6 (SW)
- new net BIND: J2.4 (Pin_4), R76.2, SW2.2, SW2.4, U2.22 (RST)
- new net HUE_RX: J2.2 (Pin_2), R70.2, U2.13 (RXD_IO7)
- new net HUE_TX: J2.3 (Pin_3), R69.1, U2.12 (TXD_IO6)
- new net PWM_1: U2.16 (IO10)
- new net PWM_B: R75.1, U2.21 (IO13)
- new net PWM_G: R73.1, U2.20 (IO12)
- new net PWM_R: R72.1, U2.19 (IO11)
